Commit message: modified:   diff_bot/urdf/caster_wheel.xacro 	new file:   diff_bot/urdf/gazebo_control.xacro 	modified:   diff_bot/urdf/properties.xacro 	modified:   diff_bot/urdf/robot.urdf.xacro modified:   diff_bot/urdf/wheels.xacro

File: diff_bot/urdf/caster_wheel.xacro (robot description, xacro)
@@ -98,3 +98,19 @@
         <child link="left_fwd_wheel_link"/>
     </joint>
+    <gazebo reference="right_back_wheel_link">
+        <mu1 value="0.01"/>
+        <mu2 value="0.01"/>
+    </gazebo>
+    <gazebo reference="left_back_wheel_link">
+        <mu1 value="0.01"/>
+        <mu2 value="0.01"/>
+    </gazebo>
+    <gazebo reference="right_fwd_wheel_link">
+        <mu1 value="0.01"/>
+        <mu2 value="0.01"/>
+    </gazebo>
+    <gazebo reference="left_fwd_wheel_link">
+        <mu1 value="0.01"/>
+        <mu2 value="0.01"/>
+    </gazebo>
 </robot>

File: diff_bot/urdf/properties.xacro (robot description, xacro)
@@ -11,5 +11,5 @@
     <xacro:property name="wheel_offset_z" value= "-0.5"/>
     <xacro:property name="wheel_thickness" value= "0.27"/>
-    <xacro:property name="wheel_radius" value= "0.325"/>
+    <xacro:property name="wheel_radius" value= "0.5"/>
     <xacro:property name="wheel_mass" value= "0.37"/>
     <!-- Caster Wheels-->
@@ -19,13 +19,13 @@
     <xacro:property name="right_back_wheel_offset_x" value= "1.9"/>
     <xacro:property name="right_back_wheel_offset_y" value= "1.4"/>
-    <xacro:property name="right_back_wheel_offset_z" value= "-0.725"/>
+    <xacro:property name="right_back_wheel_offset_z" value= "-0.4"/>
     <xacro:property name="left_back_wheel_offset_x" value= "1.9"/>
     <xacro:property name="left_back_wheel_offset_y" value= "-1.4"/>
-    <xacro:property name="left_back_wheel_offset_z" value= "-0.725"/>
+    <xacro:property name="left_back_wheel_offset_z" value= "-0.4"/>
     <xacro:property name="right_fwd_wheel_offset_x" value= "-1.9"/>
     <xacro:property name="right_fwd_wheel_offset_y" value= "1.4"/>
-    <xacro:property name="right_fwd_wheel_offset_z" value= "-0.725"/>
+    <xacro:property name="right_fwd_wheel_offset_z" value= "-0.4"/>
     <xacro:property name="left_fwd_wheel_offset_x" value= "-1.9"/>
     <xacro:property name="left_fwd_wheel_offset_y" value= "-1.4"/>
-    <xacro:property name="left_fwd_wheel_offset_z" value= "-0.725"/>
+    <xacro:property name="left_fwd_wheel_offset_z" value= "-0.4"/>
 </robot>

File: diff_bot/urdf/robot.urdf.xacro (robot description, xacro)
@@ -7,4 +7,5 @@
     <xacro:include filename="wheels.xacro"/>
     <xacro:include filename="caster_wheel.xacro"/>
+    <xacro:include filename="gazebo_control.xacro"/>
     <link name="base_link">
     </link>

File: diff_bot/urdf/wheels.xacro (robot description, xacro)
@@ -23,7 +23,7 @@
     </xacro:macro>
     <!-- wheel joint macro -->
-    <xacro:macro name="wheel_joint" params="joint_name wheel_name x_offset y_offset z_offset roll">
+    <xacro:macro name="wheel_joint" params="joint_name wheel_name x_offset y_offset z_offset">
         <joint name="${joint_name}" type="continuous">
-            <origin xyz="${x_offset} ${y_offset} ${z_offset}" rpy="${roll} 0.0 0.0"/>
+            <origin xyz="${x_offset} ${y_offset} ${z_offset}" rpy="${-pi/2} 0.0 0.0"/>
             <parent link="base_link"/>
             <child link="${wheel_name}"/>
@@ -38,8 +38,8 @@
     </xacro:wheel_link>
     <!-- left wheel joint -->
-    <xacro:wheel_joint joint_name="left_wheel_joint" wheel_name="left_wheel_link" x_offset="${wheel_offset_x}" y_offset="${wheel_offset_y}" z_offset="${wheel_offset_z}" roll="${-pi/2}">
+    <xacro:wheel_joint joint_name="left_wheel_joint" wheel_name="left_wheel_link" x_offset="${wheel_offset_x}" y_offset="${wheel_offset_y}" z_offset="${wheel_offset_z}">
     </xacro:wheel_joint>
     <!-- right wheel joint -->
-    <xacro:wheel_joint joint_name="right_wheel_joint" wheel_name="right_wheel_link" x_offset="${wheel_offset_x}" y_offset="${-wheel_offset_y}" z_offset="${wheel_offset_z}" roll="${pi/2}">
+    <xacro:wheel_joint joint_name="right_wheel_joint" wheel_name="right_wheel_link" x_offset="${wheel_offset_x}" y_offset="${-wheel_offset_y}" z_offset="${wheel_offset_z}">
     </xacro:wheel_joint>
 </robot>
