Commit message: modified:   diff_bot/urdf/properties.xacro

File: diff_bot/urdf/properties.xacro (robot description, xacro)
@@ -19,13 +19,13 @@
     <xacro:property name="right_back_wheel_offset_x" value= "1.9"/>
     <xacro:property name="right_back_wheel_offset_y" value= "1.4"/>
-    <xacro:property name="right_back_wheel_offset_z" value= "-0.4"/>
+    <xacro:property name="right_back_wheel_offset_z" value= "-0.9"/>
     <xacro:property name="left_back_wheel_offset_x" value= "1.9"/>
     <xacro:property name="left_back_wheel_offset_y" value= "-1.4"/>
-    <xacro:property name="left_back_wheel_offset_z" value= "-0.4"/>
+    <xacro:property name="left_back_wheel_offset_z" value= "-0.9"/>
     <xacro:property name="right_fwd_wheel_offset_x" value= "-1.9"/>
     <xacro:property name="right_fwd_wheel_offset_y" value= "1.4"/>
-    <xacro:property name="right_fwd_wheel_offset_z" value= "-0.4"/>
+    <xacro:property name="right_fwd_wheel_offset_z" value= "-0.9"/>
     <xacro:property name="left_fwd_wheel_offset_x" value= "-1.9"/>
     <xacro:property name="left_fwd_wheel_offset_y" value= "-1.4"/>
-    <xacro:property name="left_fwd_wheel_offset_z" value= "-0.4"/>
+    <xacro:property name="left_fwd_wheel_offset_z" value= "-0.9"/>
 </robot>
