Commit message: On branch main  Your branch is up to date with 'origin/main'.
 Changes to be committed:
	new file:   bot_nav/CMakeLists.txt
    new file:   bot_nav/config/amcl_config.yaml
    new file:   bot_nav/config/behavior.xml
	new file:   bot_nav/config/bt_navigator.yaml
	new file:   bot_nav/config/cartographer.lua
	new file:   bot_nav/config/controller.yaml
	new file:   bot_nav/config/planner_server.yaml
	new file:   bot_nav/config/recovery.yaml
	new file:   bot_nav/config/warehouse_map.pgm
	new file:   bot_nav/config/warehouse_map.yaml
	new file:   bot_nav/launch/localization.launch.py
	new file:   bot_nav/launch/mapping.launch.py
	new file:   bot_nav/launch/navigation.launch.py
	new file:   bot_nav/package.xml
	new file:   bot_nav/rviz/nav.rviz
	modified:   diff_bot/launch/robot.launch.py
	modified:   diff_bot/launch/rsp.launch.py
	modified:   diff_bot/launch/simulation.launch.py
	deleted:    diff_bot/urdf/caster_wheel.xacro
	modified:   diff_bot/urdf/chassis.xacro
	modified:   diff_bot/urdf/gazebo_control.xacro
	modified:   diff_bot/urdf/lidar.xacro
	deleted:    diff_bot/urdf/properties.xacro
	modified:   diff_bot/urdf/robot.urdf.xacro
	deleted:    diff_bot/urdf/wheels.xacro
	new file:   diff_bot/worlds/warehouse.world

File: diff_bot/urdf/chassis.xacro (robot description, xacro)
@@ -1,27 +1,238 @@
 <?xml version="1.0"?>
-<robot name="diff_bot"
-    xmlns:xacro="http://ros.org/wiki/xacro">
+<robot xmlns:xacro="http://www.ros.org/wiki/xacro" >
+    <xacro:include filename="inertial_macros.xacro"/>
+    <xacro:property name="chassis_length" value="0.7"/>
+    <xacro:property name="chassis_width" value="0.65"/>
+    <xacro:property name="chassis_height" value="0.2"/>
+    <xacro:property name="chassis_mass" value="1.0"/>
+    <xacro:property name="wheel_radius" value="0.075"/>
+    <xacro:property name="wheel_thickness" value="0.04"/>
+    <xacro:property name="wheel_mass" value="0.05"/>
+    <xacro:property name="wheel_offset_x" value="0.35"/>
+    <xacro:property name="wheel_offset_y" value="0.325"/>
+    <xacro:property name="wheel_offset_z" value="0.05"/>
+    <xacro:property name="caster_wheel_radius" value="0.05"/>
+    <xacro:property name="caster_wheel_mass" value="0.01"/>
+    <xacro:property name="right_back_wheel_offset_x" value="0.02"/>
+    <xacro:property name="left_back_wheel_offset_x" value="0.02"/>
+    <xacro:property name="right_fwd_wheel_offset_x" value="0.68"/>
+    <xacro:property name="left_fwd_wheel_offset_x" value="0.68"/>
+    <xacro:property name="right_back_wheel_offset_y" value="0.325"/>
+    <xacro:property name="left_back_wheel_offset_y" value="-0.325"/>
+    <xacro:property name="right_fwd_wheel_offset_y" value="0.325"/>
+    <xacro:property name="left_fwd_wheel_offset_y" value="-0.325"/>
+    <xacro:property name="caster_wheel_offset_z" value="${wheel_offset_z - wheel_radius + caster_wheel_radius}"/>
+    <material name="white">
+        <color rgba="1 1 1 1" />
+    </material>
+    <material name="orange">
+        <color rgba="1 0.3 0.1 1"/>
+    </material>
+    <material name="blue">
+        <color rgba="0.2 0.2 1 1"/>
+    </material>
+    <material name="black">
+        <color rgba="0 0 0 1"/>
+    </material>
+    <material name="red">
+        <color rgba="1 0 0 1"/>
+    </material>
+    <!-- BASE LINK -->
+    <link name="base_link">
+    </link>
+    <!-- BASE_FOOTPRINT LINK AND JOINT-->
+    <joint name="base_footprint_joint" type="fixed">
+        <parent link="base_link"/>
+        <child link="base_footprint"/>
+        <origin xyz="0 0 0" rpy="0 0 0"/>
+    </joint>
+    <link name="base_footprint">
+    </link>
+    <!-- CHASSIS LINK -->
+    <joint name="chassis_joint" type="fixed">
+        <parent link="base_link"/>
+        <child link="chassis_link"/>
+        <origin xyz="${-wheel_offset_x} 0 ${-wheel_offset_z}"/>
+    </joint>
     <link name="chassis_link">
         <visual>
-            <geometry>
-                <box size="4.0 3.0 1.0"/>
-                <origin xyz="2.0 0.0 0.5" rpy="0.0 0.0 0.0"/>
-            </geometry>
-        </visual>
-        <collision>
-            <geometry>
-                <box size="4.0 3.0 1.0"/>
-                <origin xyz="2.0 0.0 0.5" rpy="0.0 0.0 0.0"/>
-            </geometry>
-        </collision>
-        <xacro:inertial_box mass="2.0" x="4.0" y="3.0" z="1.0">
-            <origin xyz="2.0 0.0 0.5" rpy="0.0 0.0 0.0"/>
+            <origin xyz="${chassis_length/2} 0 ${chassis_height/2}"/>
+            <geometry>
+                <box size="${chassis_length} ${chassis_width} ${chassis_height}"/>
+            </geometry>
+            <material name="orange"/>
+        </visual>
+        <collision>
+            <origin xyz="${chassis_length/2} 0 ${chassis_height/2}"/>
+            <geometry>
+                <box size="${chassis_length} ${chassis_width} ${chassis_height}"/>
+            </geometry>
+        </collision>
+        <xacro:inertial_box mass="0.5" x="${chassis_length}" y="${chassis_width}" z="${chassis_height}">
+            <origin xyz="${chassis_length/2} 0 ${chassis_height/2}" rpy="0 0 0"/>
         </xacro:inertial_box>
     </link>
-    <!-- Chassis joint -->
-    <joint name="chassis_joint" type="fixed">
-        <parent link="base_link"/>
-        <child link="chassis_link"/>
-        <origin xyz="-2.0 0.0 0.0" rpy="0.0 0.0 0.0"/>
-    </joint>
+    <gazebo reference="chassis_link">
+        <material>Gazebo/Orange</material>
+    </gazebo>
+    <!-- LEFT WHEEL LINK -->
+    <joint name="left_wheel_joint" type="continuous">
+        <parent link="base_link"/>
+        <child link="left_wheel"/>
+        <origin xyz="0 ${wheel_offset_y} 0" rpy="-${pi/2} 0 0" /> <!-- rotating the axes of cylinder from default mode to make axis of rotation normal to the chassis-->
+        <axis xyz="0 0 1"/> <!-- determining the axis of rotation to the wheel about z axis -->
+    </joint>
+    <link name="left_wheel">
+        <visual>
+            <geometry>
+                <cylinder radius="${wheel_radius}" length="${wheel_thickness}"/>
+            </geometry>
+            <material name="blue"/>
+        </visual>
+        <collision>
+            <geometry>
+                <sphere radius="${wheel_radius}"/>
+            </geometry>
+        </collision>
+        <xacro:inertial_cylinder mass="${wheel_mass}" length="${wheel_thickness}" radius="${wheel_radius}">
+            <origin xyz="0 0 0" rpy="0 0 0"/>
+        </xacro:inertial_cylinder>
+    </link>
+    <gazebo reference="left_wheel">
+        <material>Gazebo/Blue</material>
+    </gazebo>
+    <!-- RIGHT WHEEL LINK -->
+    <joint name="right_wheel_joint" type="continuous">
+        <parent link="base_link"/>
+        <child link="right_wheel"/>
+        <origin xyz="0 ${-wheel_offset_y} 0" rpy="${pi/2} 0 0" />
+        <axis xyz="0 0 -1"/>
+    </joint>
+    <link name="right_wheel">
+        <visual>
+            <geometry>
+                <cylinder radius="${wheel_radius}" length="${wheel_thickness}"/>
+            </geometry>
+            <material name="blue"/>
+        </visual>
+        <collision>
+            <geometry>
+                <sphere radius="${wheel_radius}"/>
+            </geometry>
+        </collision>
+        <xacro:inertial_cylinder mass="${wheel_mass}" length="${wheel_thickness}" radius="${wheel_radius}">
+            <origin xyz="0 0 0" rpy="0 0 0"/>
+        </xacro:inertial_cylinder>
+    </link>
+    <gazebo reference="right_wheel">
+        <material>Gazebo/Blue</material>
+    </gazebo>
+    <!-- RIGHT_BACK WHEEL LINK -->
+    <joint name="right_back_wheel_joint" type="fixed">
+        <parent link="chassis_link"/>
+        <child link="right_back_wheel"/>
+        <origin xyz="${right_back_wheel_offset_x} ${right_back_wheel_offset_y} ${caster_wheel_offset_z}"/>
+    </joint>
+    <link name="right_back_wheel">
+        <visual>
+            <geometry>
+                <sphere radius="${caster_wheel_radius}"/>
+            </geometry>
+            <material name="white"/>
+        </visual>
+        <collision>
+            <geometry>
+                <sphere radius="${caster_wheel_radius}"/>
+            </geometry>
+        </collision>
+        <xacro:inertial_sphere mass="${caster_wheel_mass}" radius="${caster_wheel_radius}">
+            <origin xyz="0 0 0" rpy="0 0 0"/>
+        </xacro:inertial_sphere>
+    </link>
+        <!-- LEFT_BACK WHEEL LINK -->
+        <joint name="left_back_wheel_joint" type="fixed">
+            <parent link="chassis_link"/>
+            <child link="left_back_wheel"/>
+            <origin xyz="${left_back_wheel_offset_x} ${left_back_wheel_offset_y} ${caster_wheel_offset_z}"/>
+        </joint>
+        <link name="left_back_wheel">
+            <visual>
+                <geometry>
+                    <sphere radius="${caster_wheel_radius}"/>
+                </geometry>
+                <material name="white"/>
+            </visual>
+            <collision>
+                <geometry>
+                    <sphere radius="${caster_wheel_radius}"/>
+                </geometry>
+            </collision>
+            <xacro:inertial_sphere mass="${caster_wheel_mass}" radius="${caster_wheel_radius}">
+                <origin xyz="0 0 0" rpy="0 0 0"/>
+            </xacro:inertial_sphere>
+        </link>
+        <!-- RIGHT_FWD WHEEL LINK -->
+        <joint name="right_fwd_wheel_joint" type="fixed">
+            <parent link="chassis_link"/>
+            <child link="right_fwd_wheel"/>
+            <origin xyz="${right_fwd_wheel_offset_x} ${right_fwd_wheel_offset_y} ${caster_wheel_offset_z}"/>
+        </joint>
+        <link name="right_fwd_wheel">
+            <visual>
+                <geometry>
+                    <sphere radius="${caster_wheel_radius}"/>
+                </geometry>
+                <material name="white"/>
+            </visual>
+            <collision>
+                <geometry>
+                    <sphere radius="${caster_wheel_radius}"/>
+                </geometry>
+            </collision>
+            <xacro:inertial_sphere mass="${caster_wheel_mass}" radius="${caster_wheel_radius}">
+            <origin xyz="0 0 0" rpy="0 0 0"/>
+            </xacro:inertial_sphere>
+        </link>
+        <!-- LEFT_FWD WHEEL LINK -->
+        <joint name="left_fwd_wheel_joint" type="fixed">
+            <parent link="chassis_link"/>
+            <child link="left_fwd_wheel"/>
+            <origin xyz="${left_fwd_wheel_offset_x} ${left_fwd_wheel_offset_y} ${caster_wheel_offset_z}"/>
+        </joint>
+        <link name="left_fwd_wheel">
+            <visual>
+                <geometry>
+                    <sphere radius="${caster_wheel_radius}"/>
+                </geometry>
+                <material name="white"/>
+            </visual>
+            <collision>
+                <geometry>
+                    <sphere radius="${caster_wheel_radius}"/>
+                </geometry>
+            </collision>
+            <xacro:inertial_sphere mass="${caster_wheel_mass}" radius="${caster_wheel_radius}">
+                <origin xyz="0 0 0" rpy="0 0 0"/>
+            </xacro:inertial_sphere>
+        </link>
+    <gazebo reference="right_back_wheel">
+        <material>Gazebo/White</material>
+        <mu1 value="0.001"/>
+        <mu2 value="0.001"/>
+    </gazebo>
+    <gazebo reference="left_back_wheel">
+        <material>Gazebo/White</material>
+        <mu1 value="0.001"/>
+        <mu2 value="0.001"/>
+    </gazebo>
+    <gazebo reference="right_fwd_wheel">
+        <material>Gazebo/White</material>
+        <mu1 value="0.001"/>
+        <mu2 value="0.001"/>
+    </gazebo>
+    <gazebo reference="left_fwd_wheel">
+        <material>Gazebo/White</material>
+        <mu1 value="0.001"/>
+        <mu2 value="0.001"/>
+    </gazebo>
 </robot>

File: diff_bot/urdf/gazebo_control.xacro (robot description, xacro)
@@ -6,5 +6,5 @@
             <right_joint>right_wheel_joint</right_joint>
             <wheel_separation>${chassis_width}</wheel_separation>
-            <wheel_diameter>0.065</wheel_diameter>
+            <wheel_diameter>0.15</wheel_diameter>
             <max_wheel_torque>200</max_wheel_torque>
             <max_wheel_acceleration>3.0</max_wheel_acceleration>

File: diff_bot/urdf/lidar.xacro (robot description, xacro)
@@ -16,5 +16,5 @@
     </gazebo>
     <joint name="laser_joint" type="fixed">
-        <origin xyz="0.07 0.0 0.18" rpy="0.0 0.0 0.0"/>
+        <origin xyz="0.122 0.0 0.25" rpy="0.0 0.0 0.0"/>
         <parent link="chassis_link"/>
         <child link="laser_frame"/>

File: diff_bot/urdf/robot.urdf.xacro (robot description, xacro)
@@ -2,13 +2,7 @@
 <robot name="diff_bot"
        xmlns:xacro="http://ros.org/wiki/xacro">
-    <xacro:include filename="properties.xacro"/>
-    <xacro:include filename="inertial_macros.xacro"/>
     <xacro:include filename="chassis.xacro"/>
-    <xacro:include filename="wheels.xacro"/>
-    <xacro:include filename="caster_wheel.xacro"/>
     <xacro:include filename="gazebo_control.xacro"/>
     <xacro:include filename="control.xacro"/>
     <xacro:include filename="lidar.xacro"/>
-    <link name="base_link">
-    </link>
 </robot>
